File: Boards/GP2040-CE Official Boards/RP2350 Duel/_restore_backup_2026-07-11T19-11-06-914/RP2350 Duel.kicad_sch (KiCad schematic)
At the start: 28 parts, among them U1 W25Q128JVS, U2 RP2350B

Commit message: Add fp-lib-table for GP2040-CE and RP2350 Duel libraries
- Created a new fp-lib-table file to include the GP2040-CE_Library and RP2350Duel libraries.
- Specified library URIs and types for integration with KiCad.
Parts:
- U2: footprint RP2350Duel:QFN-80-1EP_10x10mm_P0.4mm_EP3.4x3.4mm -> Package_DFN_QFN:QFN-80-1EP_10x10mm_P0.4mm_EP3.4x3.4mm
- Y1: renamed from G1; value SiT8008BI-72-33N-12.000000 -> SiT8008xx-7x-xxE; footprint RP2350Duel:OSC_SiT8008BI-72-33N-12.000000 -> Oscillator:Oscillator_SMD_SiT_PQFN-4Pin_2.0x1.6mm; symbol RP2350Duel:SiT8008BI-72-33N-12.000000 -> Oscillator:SiT8008xx-7x-xxE; CREATOR ASHISH -> (none); MANUFACTURER SiTime -> (none); MAXIMUM_PACKAGE_HEIGHT 0.8mm -> (none); PARTREV 1.08 -> (none); STANDARD Manufacturer Recommendations -> (none)
Connections:
- net +1V1: now also R2.1, Y1.4 (Vdd)
- net +3.3V: no longer R2.1
- net GND: no longer U3.1 (GND), U3.11 (GND), U3.15 (GND), U3.21 (GND), U3.4 (GND), U3.7 (GND)
- net at Y1.1 (OE): now also R2.2
- net USB_DN renamed USB_DM
- new net: U3.1 (GND), U3.11 (GND), U3.15 (GND), U3.21 (GND), U3.4 (GND), U3.7 (GND)
Other:
- sheet Power ports: added none; removed DM, DP
