File: Boards/GP2040-CE Official Boards/RP2350 Duel/Power.kicad_sch (KiCad schematic)
At the start: 13 parts, among them J1 UJ20-C-H-G-SMT-2A-P16-TR, U4 TVS2200DRV, U5 24LC512, U6 TPD4EUSB30, U7 TPS25751SRSMR

Commit message: Refactor code structure for improved readability and maintainability
Parts:
- U5: footprint (none) -> RP2350Duel:24LC512
- U7: footprint TPS25751SRSMR:RSM0032B-IPC_A -> RP2350Duel:RSM0032B-MFG
Connections:
- net GND: now also U7.11 (GND), U7.12 (GND), U7.14 (GND)
- no-connect marks 9 -> 18
Changed lines of the file:
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@@
+	)
+	(junction
+		(at 190.5 92.71)
+		(diameter 0)
+		(color 0 0 0 0)
+	)
+	(junction
+		(at 190.5 90.17)
+		(diameter 0)
+		(color 0 0 0 0)
 	)
 	(junction
@@
 		(color 0 0 0 0)
 	)
+	(junction
+		(at 190.5 87.63)
+		(diameter 0)
+		(color 0 0 0 0)
+	)
 	(no_connect
 		(at 46.99 64.77)
@@
 	)
 	(no_connect
+		(at 190.5 36.83)
+	)
+	(no_connect
 		(at 83.82 77.47)
 	)
@@
 	)
 	(no_connect
+		(at 190.5 29.21)
+	)
+	(no_connect
+		(at 190.5 41.91)
+	)
+	(no_connect
+		(at 190.5 31.75)
+	)
+	(no_connect
+		(at 190.5 46.99)
+	)
+	(no_connect
+		(at 190.5 49.53)
+	)
+	(no_connect
+		(at 190.5 44.45)
+	)
+	(no_connect
 		(at 83.82 80.01)
 	)
+	(no_connect
+		(at 190.5 34.29)
+	)
+	(no_connect
+		(at 190.5 39.37)
+	)
 	(wire
 		(pts
@@
 	(wire
 		(pts
+			(xy 190.5 87.63) (xy 190.5 90.17)
+		)
+		(stroke
+			(width 0)
+			(type default)
+		)
+	)
+	(wire
+		(pts
 			(xy 134.62 87.63) (xy 123.19 87.63)
 		)
@@
 	(wire
 		(pts
+			(xy 190.5 90.17) (xy 190.5 92.71)
+		)
+		(stroke
+			(width 0)
+			(type default)
+		)
+	)
+	(wire
+		(pts
 			(xy 77.47 67.31) (xy 88.9 67.31)
 		)
@@
 		(pts
 			(xy 119.38 45.72) (xy 134.62 45.72)
+		)
+		(stroke
+			(width 0)
+			(type default)
+		)
+	)
+	(wire
+		(pts
+			(xy 190.5 85.09) (xy 190.5 87.63)
 		)
 		(stroke
@@
 			)
 		)
-		(property "Footprint" ""
+		(property "Footprint" "RP2350Duel:24LC512"
 			(at 93.98 80.01 0)
 			(hide yes)
@@
 			)
 		)
-		(property "Footprint" "TPS25751SRSMR:RSM0032B-IPC_A"
+		(property "Footprint" "RP2350Duel:RSM0032B-MFG"
 			(at 134.62 29.21 0)
 			(hide yes)
