File: Boards/GP2040-CE Official Boards/RP2350 Duel/RP2350 Duel.kicad_pcb (KiCad board)
At the start: 4 copper layers, 79.5 x 64.5 mm, 41 parts, among them J1 UJ20-C-H-G-SMT-2A-P16-TR, U1 W25Q128JVS, U2 RP2350B, U4 TVS2200DRV, U6 TPD4EUSB30, U7 TPS25751SRSMR

Commit message: Refactor code structure for improved readability and maintainability
Parts:
- added U5: 24LC512, RP2350Duel:24LC512, F.Cu at (143.0, 66.8)
- L1: footprint MLZ2012M3R3HT000:IND_2012_TDK -> RP2350Duel:IND_2012_TDK
- L2: footprint BLM18EG471SN1D:IND_BLM18_0603_MUR -> RP2350Duel:IND_BLM18_0603_MUR
- U7: footprint TPS25751SRSMR:RSM0032B-IPC_A -> RP2350Duel:RSM0032B-MFG
- moved R1 119.5 mm to (131.3, 74.7), turned to -90 degrees
- moved R2 92.7 mm to (157.5, 71.1)
- moved R3 92.5 mm to (157.5, 72.6), turned to 180 degrees
- moved R6 91.8 mm to (157.5, 74.2)
- moved C15 89.4 mm to (138.4, 71.9), turned to 180 degrees
- moved C10 79.8 mm to (142.5, 79.0), turned to 180 degrees
- moved C11 77.4 mm to (151.4, 71.4), turned to 90 degrees
- moved C7 77.3 mm to (142.5, 77.5), turned to 180 degrees
- moved C2 73.1 mm to (142.5, 80.5), turned to 180 degrees
- moved C1 71.3 mm to (147.8, 71.4), turned to 90 degrees
- moved C16 71.1 mm to (160.8, 72.6)
- moved R8 70.9 mm to (148.6, 65.8)
- moved C14 69.6 mm to (157.5, 75.7)
- moved C12 68.9 mm to (160.8, 75.7)
- moved C9 68.4 mm to (150.6, 86.4), turned to -90 degrees
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Connections:
- net /USB_DM renamed /USB_DN
- U7 pad 11: unconnected-(U7-GND-Pad11) -> GND
- U7 pad 12: unconnected-(U7-GND-Pad12) -> GND
- U7 pad 14: unconnected-(U7-GND-Pad14) -> GND
Routing:
- net /WL_D: track 48.2 -> 0.00 mm, vias 2 -> 0
- net /Power/VBUS: track 24.9 -> 0.00 mm
- net GND: track 12.8 -> 0.00 mm, vias 1 -> 0
- net /Power/D-: track 11.0 -> 0.00 mm, vias 3 -> 0
- net /Power/D+: track 10.8 -> 0.00 mm, vias 3 -> 0
- net /gSPI_Data_In: track 9.76 -> 0.00 mm
- net /Power/CC1: track 9.60 -> 0.00 mm
- net /Power/CC2: track 8.82 -> 0.00 mm
- net /VDDIO: track 8.69 -> 0.00 mm
- net +3.3V: track 3.82 -> 0.00 mm, vias 3 -> 0
- net /XIN: track 3.62 -> 0.00 mm
- net /nIRQ: track 3.14 -> 0.00 mm
- net /WL_ON: track 1.50 -> 0.00 mm
- added copper zone on In2.Cu, net +1V1

Commit message: new footprints
Parts:
- removed the R2 at (157.5, 71.1)
- added J2: Conn_02x08_Odd_Even, RP2350Duel:FlexPCB, F.Cu at (114.6, 72.1)
- added SW1: SW_SPST, RP2350Duel:SKRWAEE030, F.Cu at (104.7, 57.8)
- added SW2: SW_SPST, RP2350Duel:SKRWAEE030, F.Cu at (172.2, 57.8)
- added SW3: SW_SPST, RP2350Duel:SKRWAEE030, F.Cu at (138.2, 102.3)
- moved C17 46.9 mm to (179.0, 100.0)
- moved R8 46.9 mm to (179.0, 101.5)
- moved C1 46.8 mm to (184.0, 101.0)
- moved C19 46.6 mm to (181.5, 77.5)
- moved C20 46.6 mm to (181.5, 79.0)
- moved U3 44.0 mm to (150.2, 84.8), turned to 180 degrees
- moved C10 43.1 mm to (184.0, 90.5)
- moved C2 43.1 mm to (184.0, 92.0)
- moved C7 43.1 mm to (184.0, 89.0)
- moved R7 40.2 mm to (179.5, 84.0)
- moved R1 40.2 mm to (171.4, 77.3)
- moved G1 36.8 mm to (176.0, 66.5)
- moved C18 35.7 mm to (178.8, 63.0)
- moved C21 35.7 mm to (182.9, 62.8)
- moved C22 35.7 mm to (179.0, 61.5)
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Connections:
- U2 pad 1: unconnected-(U2-GPIO4-Pad1) -> /RIGHT
- U2 pad 11: unconnected-(U2-GPIO12-Pad11) -> /R1
- U2 pad 12: unconnected-(U2-GPIO13-Pad12) -> /L1
- U2 pad 16: unconnected-(U2-GPIO16-Pad16) -> /SELECT
- U2 pad 17: unconnected-(U2-GPIO17-Pad17) -> /START
- U2 pad 18: unconnected-(U2-GPIO18-Pad18) -> /L3
- U2 pad 19: unconnected-(U2-GPIO19-Pad19) -> /R3
- U2 pad 2: unconnected-(U2-GPIO5-Pad2) -> /LEFT
- U2 pad 20: unconnected-(U2-GPIO20-Pad20) -> /MUTE
- U2 pad 3: unconnected-(U2-GPIO6-Pad3) -> /X
- U2 pad 4: unconnected-(U2-GPIO7-Pad4) -> /CIR
- U2 pad 6: unconnected-(U2-GPIO8-Pad6) -> /R2
- U2 pad 7: unconnected-(U2-GPIO9-Pad7) -> /L2
- U2 pad 79: unconnected-(U2-GPIO2-Pad79) -> /UP
- U2 pad 8: unconnected-(U2-GPIO10-Pad8) -> /SQ
- U2 pad 80: unconnected-(U2-GPIO3-Pad80) -> /DOWN
- U2 pad 9: unconnected-(U2-GPIO11-Pad9) -> /TR

Commit message: updating boards
Parts:
- moved R5 51.4 mm to (209.6, 70.4)
- moved C15 51.3 mm to (209.6, 71.3)
- moved U1 47.8 mm to (120.1, 63.2)
- moved R2 41.8 mm to (208.6, 73.2)
- moved C11 39.9 mm to (208.6, 82.5)
- moved U3 37.9 mm to (167.2, 50.8), turned to -5.5 degrees
- moved R1 37.2 mm to (208.6, 76.9)
- moved C5 34.9 mm to (209.6, 100.2)
- moved C6 34.8 mm to (209.6, 101.1)
- moved R3 34.7 mm to (209.6, 84.3)
- moved R6 34.6 mm to (209.6, 88.1)
- moved C8 34.6 mm to (209.6, 93.7)
- moved C4 34.6 mm to (209.6, 92.7)
- moved C14 34.6 mm to (209.6, 90.9)
- moved R4 33.0 mm to (209.6, 75.0)
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Connections:
- U2 pad 1: /RIGHT -> /LEFT
- U2 pad 11: /R1 -> /CIR
- U2 pad 12: /L1 -> /X
- U2 pad 13: unconnected-(U2-GPIO14-Pad13) -> /PS
- U2 pad 2: /LEFT -> /UP
- U2 pad 3: /X -> /L1
- U2 pad 4: /CIR -> /L2
- U2 pad 7: /L2 -> /R1
- U2 pad 79: /UP -> /DOWN
- U2 pad 80: /DOWN -> /RIGHT
Routing:
- net /SELECT: track 0.00 -> 45.8 mm, vias 0 -> 2
- net /DOWN: track 0.00 -> 36.8 mm
- net /RIGHT: track 0.00 -> 34.3 mm
- net /MUTE: track 0.00 -> 32.9 mm, vias 0 -> 2
- net /UP: track 0.00 -> 29.9 mm
- net /LEFT: track 0.00 -> 28.5 mm
- net /L2: track 0.00 -> 25.3 mm
- net /L1: track 0.00 -> 25.0 mm
- net /R2: track 0.00 -> 23.5 mm
- net GND: track 0.00 -> 21.0 mm, vias 0 -> 3
- net /Power/VBUS: track 0.00 -> 20.8 mm
- net /R1: track 0.00 -> 20.0 mm
- net /TR: track 0.00 -> 19.9 mm
- net /SQ: track 0.00 -> 18.5 mm
- net /Power/CC1: track 0.00 -> 15.7 mm, vias 0 -> 2
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- added copper zone on In1.Cu, net GND
