File: Boards/GP2040-CE Official Boards/RP2350 Duel/RP2350 Duel.kicad_sch (KiCad schematic)
At the start: 28 parts, among them U1 W25Q128JVS, U2 RP2350B

Commit message: Refactor code structure for improved readability and maintainability
Parts:
- added J2: Conn_02x08_Odd_Even, symbol Connector_Generic:Conn_02x08_Odd_Even
- L1: footprint MLZ2012M3R3HT000:IND_2012_TDK -> RP2350Duel:IND_2012_TDK
- L2: footprint BLM18EG471SN1D:IND_BLM18_0603_MUR -> RP2350Duel:IND_BLM18_0603_MUR
Changed lines of the file:
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@@
 			)
 		)
-		(property "Footprint" "MLZ2012M3R3HT000:IND_2012_TDK"
+		(property "Footprint" "RP2350Duel:IND_2012_TDK"
 			(at 196.85 44.45 0)
 			(hide yes)
@@
 	)
 	(symbol
+		(lib_id "Connector_Generic:Conn_02x08_Odd_Even")
+		(at 186.69 116.84 0)
+		(unit 1)
+		(body_style 1)
+		(exclude_from_sim no)
+		(in_bom yes)
+		(on_board yes)
+		(in_pos_files yes)
+		(dnp no)
+		(fields_autoplaced yes)
+		(property "Reference" "J2"
+			(at 187.96 102.87 0)
+			(show_name no)
+			(do_not_autoplace no)
+			(effects
+				(font
+					(size 1.27 1.27)
+				)
+			)
+		)
+		(property "Value" "Conn_02x08_Odd_Even"
+			(at 187.96 105.41 0)
+			(show_name no)
+			(do_not_autoplace no)
+			(effects
+				(font
+					(size 1.27 1.27)
+				)
+			)
+		)
+		(property "Footprint" ""
+			(at 186.69 116.84 0)
+			(hide yes)
+			(show_name no)
+			(do_not_autoplace no)
+			(effects
+				(font
+					(size 1.27 1.27)
+				)
+			)
+		)
+		(property "Datasheet" ""
+			(at 186.69 116.84 0)
+			(hide yes)
+			(show_name no)
+			(do_not_autoplace no)
+			(effects
+				(font
+					(size 1.27 1.27)
+				)
+			)
+		)
+		(property "Description" "Generic connector, double row, 02x08, odd/even pin numbering scheme (row 1 odd numbers, row 2 even numbers), script generated (kicad-library-utils/schlib/autogen/connector/)"
+			(at 186.69 116.84 0)
+			(hide yes)
+			(show_name no)
+			(do_not_autoplace no)
+			(effects
+				(font
+					(size 1.27 1.27)
+				)
+			)
+		)
+		(pin "2"
+		)
+		(pin "12"
+		)
+		(pin "1"
+		)
+		(pin "3"
+		)
+		(pin "4"
+		)
+		(pin "5"
+		)
+		(pin "6"
+		)
+		(pin "7"
+		)
+		(pin "8"
+		)
+		(pin "9"
+		)
+		(pin "10"
+		)
+		(pin "11"
+		)
+		(pin "16"
+		)
+		(pin "14"
+		)
+		(pin "13"
+		)
+		(pin "15"
+		)
+		(instances
+			(project "RP2350 Duel"
+				(path "/9569aed4-f877-407f-b337-4ee93294723e"
+					(reference "J2")
+					(unit 1)
+				)
+			)
+		)
+	)
+	(symbol
 		(lib_id "Device:C_Small")
 		(at 25.4 81.28 0)
@@
 			)
 		)
-		(property "Footprint" "BLM18EG471SN1D:IND_BLM18_0603_MUR"
+		(property "Footprint" "RP2350Duel:IND_BLM18_0603_MUR"
 			(at 240.03 107.95 0)
 			(hide yes)

Commit message: new footprints
Parts:
- added SW1, SW2, SW3: SW_SPST, RP2350Duel:SKRWAEE030, symbol Switch:SW_SPST
- J2: footprint (none) -> RP2350Duel:FlexPCB
Connections:
- net GND: now also J2.11 (Pin_11), J2.2 (Pin_2), SW1.2 (B), SW2.2 (B), SW3.2 (B)
- net DOWN: now reaches J2.1 (Pin_1)
- net DOWN: now also U2.80 (GPIO3)
- net R1: now reaches J2.10 (Pin_10)
- net R1: now also U2.11 (GPIO12)
- net SQ: now reaches J2.12 (Pin_12)
- net SQ: now also U2.8 (GPIO10)
- net TR: now reaches J2.13 (Pin_13)
- net TR: now also U2.9 (GPIO11)
- net CIR: now reaches J2.14 (Pin_14)
- net CIR: now also U2.4 (GPIO7)
- net X: now reaches J2.15 (Pin_15)
- net X: now also U2.3 (GPIO6)
- net PS: now reaches J2.16 (Pin_16)
- net RIGHT: now reaches J2.3 (Pin_3)
- net RIGHT: now also U2.1 (GPIO4)
- net LEFT: now reaches J2.4 (Pin_4)
- net LEFT: now also U2.2 (GPIO5)
- net UP: now reaches J2.5 (Pin_5)
- net UP: now also U2.79 (GPIO2)
- net L1: now reaches J2.6 (Pin_6)
- net L1: now also U2.12 (GPIO13)
- net L2: now reaches J2.7 (Pin_7)
- net L2: now also U2.7 (GPIO9)
- net R2: now reaches J2.9 (Pin_9)
- net R2: now also U2.6 (GPIO8)
- net SELECT: now reaches U2.16 (GPIO16)
- net SELECT: now also SW1.1 (A)
- net START: now reaches U2.17 (GPIO17)
- net START: now also SW2.1 (A)
- net L3: now reaches U2.18 (GPIO18)
- net R3: now reaches U2.19 (GPIO19)
- net MUTE: now reaches U2.20 (GPIO20)
- net MUTE: now also SW3.1 (A)
- no-connect marks 0 -> 1

Commit message: updating boards
Connections:
- net CIR: now also U2.11 (GPIO12); no longer U2.4 (GPIO7)
- net DOWN: now also U2.79 (GPIO2); no longer U2.80 (GPIO3)
- net L1: now also U2.3 (GPIO6); no longer U2.12 (GPIO13)
- net L2: now also U2.4 (GPIO7); no longer U2.7 (GPIO9)
- net LEFT: now also U2.1 (GPIO4); no longer U2.2 (GPIO5)
- net PS: now also U2.13 (GPIO14)
- net R1: now also U2.7 (GPIO9); no longer U2.11 (GPIO12)
- net RIGHT: now also U2.80 (GPIO3); no longer U2.1 (GPIO4)
- net UP: now also U2.2 (GPIO5); no longer U2.79 (GPIO2)
- net X: now also U2.12 (GPIO13); no longer U2.3 (GPIO6)
Changed lines of the file:
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@@
+		)
+	)
+	(label "CIR"
+		(at 78.74 63.5 180)
+		(effects
+			(font
+				(size 1.27 1.27)
+			)
+			(justify right bottom)
+		)
+	)
+	(label "VDDIO"
+		(at 257.81 74.93 0)
+		(effects
+			(font
+				(size 1.27 1.27)
+			)
+			(justify left bottom)
+		)
+	)
+	(label "VREG_FB"
+		(at 132.08 30.48 90)
+		(effects
+			(font
+				(size 1.27 1.27)
+			)
+			(justify left bottom)
+		)
+	)
+	(label "VREG_AVDD"
+		(at 204.47 29.21 0)
+		(effects
+			(font
+				(size 1.27 1.27)
+			)
+			(justify left bottom)
+		)
+	)
+	(label "RIGHT"
+		(at 93.98 30.48 90)
+		(effects
+			(font
+				(size 1.27 1.27)
+			)
+			(justify left bottom)
+		)
+	)
+	(label "L1"
+		(at 194.31 114.3 0)
+		(effects
+			(font
+				(size 1.27 1.27)
+			)
+			(justify left bottom)
+		)
+	)
+	(label "START"
+		(at 78.74 78.74 180)
+		(effects
+			(font
+				(size 1.27 1.27)
+			)
+			(justify right bottom)
+		)
+	)
+	(label "gSPI_CS"
+		(at 105.41 96.52 270)
+		(effects
+			(font
+				(size 1.27 1.27)
+			)
+			(justify right bottom)
+		)
+	)
+	(label "ADC_VREF"
+		(at 213.36 25.4 180)
+		(effects
+			(font
+				(size 1.27 1.27)
+			)
+			(justify right bottom)
+		)
+	)
+	(label "USB_DP"
+		(at 127 30.48 90)
+		(effects
+			(font
+				(size 1.27 1.27)
+			)
+			(justify left bottom)
+		)
+	)
+	(label "ADC_AVDD"
+		(at 48.26 106.68 180)
+		(effects
+			(font
+				(size 1.27 1.27)
+			)
+			(justify right bottom)
+		)
+	)
+	(label "IOVDD"
+		(at 62.23 24.13 180)
+		(effects
+			(font
+				(size 1.27 1.27)
+			)
+			(justify right bottom)
 		)
 	)
@@
 		)
 	)
-	(label "VDDIO"
-		(at 257.81 74.93 0)
-		(effects
-			(font
-				(size 1.27 1.27)
-			)
-			(justify left bottom)
-		)
-	)
-	(label "VREG_FB"
-		(at 132.08 30.48 90)
-		(effects
-			(font
-				(size 1.27 1.27)
-			)
-			(justify left bottom)
-		)
-	)
-	(label "VREG_AVDD"
-		(at 204.47 29.21 0)
-		(effects
-			(font
-				(size 1.27 1.27)
-			)
-			(justify left bottom)
-		)
-	)
-	(label "L1"
-		(at 194.31 114.3 0)
-		(effects
-			(font
-				(size 1.27 1.27)
-			)
-			(justify left bottom)
-		)
-	)
-	(label "START"
-		(at 78.74 78.74 180)
-		(effects
-			(font
-				(size 1.27 1.27)
-			)
-			(justify right bottom)
-		)
-	)
-	(label "gSPI_CS"
-		(at 105.41 96.52 270)
-		(effects
-			(font
-				(size 1.27 1.27)
-			)
-			(justify right bottom)
-		)
-	)
-	(label "ADC_VREF"
-		(at 213.36 25.4 180)
-		(effects
-			(font
-				(size 1.27 1.27)
-			)
-			(justify right bottom)
-		)
-	)
-	(label "USB_DP"
-		(at 127 30.48 90)
-		(effects
-			(font
-				(size 1.27 1.27)
-			)
-			(justify left bottom)
-		)
-	)
-	(label "ADC_AVDD"
-		(at 48.26 106.68 180)
-		(effects
-			(font
-				(size 1.27 1.27)
-			)
-			(justify right bottom)
-		)
-	)
-	(label "IOVDD"
-		(at 62.23 24.13 180)
+	(label "PS"
+		(at 78.74 68.58 180)
 		(effects
 			(font
@@
 		)
 	)
-	(label "RIGHT"
-		(at 78.74 38.1 180)
-		(effects
-			(font
-				(size 1.27 1.27)
-			)
-			(justify right bottom)
-		)
-	)
 	(label "SELECT"
 		(at 217.17 119.38 180)
@@
 		)
 	)
+	(label "R2"
+		(at 78.74 50.8 180)
+		(effects
+			(font
+				(size 1.27 1.27)
+			)
+			(justify right bottom)
+		)
+	)
 	(label "R3"
 		(at 78.74 83.82 180)
@@
 		)
 	)
-	(label "L1"
-		(at 78.74 66.04 180)
-		(effects
-			(font
-				(size 1.27 1.27)
-			)
-			(justify right bottom)
-		)
-	)
 	(label "VREG_VIN"
 		(at 46.99 92.71 180)
@@
 		)
 	)
-	(label "DOWN"
-		(at 93.98 30.48 90)
-		(effects
-			(font
-				(size 1.27 1.27)
-			)
-			(justify left bottom)
-		)
-	)
 	(label "VREG_VIN"
 		(at 254 25.4 0)
@@
 		)
 	)
+	(label "L1"
+		(at 78.74 43.18 180)
+		(effects
+			(font
+				(size 1.27 1.27)
+			)
+			(justify right bottom)
+		)
+	)
 	(label "SQ"
 		(at 194.31 121.92 0)
@@
 		)
 	)
+	(label "DOWN"
+		(at 96.52 30.48 90)
+		(effects
+			(font
+				(size 1.27 1.27)
+			)
+			(justify left bottom)
+		)
+	)
+	(label "X"
+		(at 78.74 66.04 180)
+		(effects
+			(font
+				(size 1.27 1.27)
+			)
+			(justify right bottom)
+		)
+	)
 	(label "USB_DN"
 		(at 129.54 30.48 90)
@@
 		)
 	)
+	(label "L2"
+		(at 78.74 45.72 180)
+		(effects
+			(font
+				(size 1.27 1.27)
+			)
+			(justify right bottom)
+		)
+	)
 	(label "gSPI_Data_In"
 		(at 215.9 72.39 180)
@@
 		)
 	)
-	(label "R2"
-		(at 78.74 50.8 180)
-		(effects
-			(font
-				(size 1.27 1.27)
-			)
-			(justify right bottom)
-		)
-	)
 	(label "VREG_FB"
 		(at 45.72 64.77 180)
@@
 		)
 	)
+	(label "LEFT"
+		(at 78.74 38.1 180)
+		(effects
+			(font
+				(size 1.27 1.27)
+			)
+			(justify right bottom)
+		)
+	)
 	(label "nIRQ"
 		(at 238.76 82.55 270)
@@
 		)
 	)
-	(label "L2"
-		(at 78.74 53.34 180)
-		(effects
-			(font
-				(size 1.27 1.27)
-			)
-			(justify right bottom)
-		)
-	)
 	(label "VDDIO"
 		(at 248.92 82.55 270)
@@
 		)
 	)
-	(label "CIR"
-		(at 78.74 45.72 180)
-		(effects
-			(font
-				(size 1.27 1.27)
-			)
-			(justify right bottom)
-		)
-	)
 	(label "IOVDD"
 		(at 78.74 73.66 180)
@@
 		)
 	)
-	(label "LEFT"
-		(at 78.74 40.64 180)
-		(effects
-			(font
-				(size 1.27 1.27)
-			)
-			(justify right bottom)
-		)
-	)
 	(label "QSPI_SD0"
 		(at 16.51 138.43 0)
@@
 		)
 	)
+	(label "SQ"
+		(at 78.74 55.88 180)
+		(effects
+			(font
+				(size 1.27 1.27)
+			)
+			(justify right bottom)
+		)
+	)
 	(label "USB_DP"
 		(at 118.11 142.24 0)
@@
 		)
 	)
+	(label "R1"
+		(at 78.74 53.34 180)
+		(effects
+			(font
+				(size 1.27 1.27)
+			)
+			(justify right bottom)
+		)
+	)
 	(label "QSPI_IOVDD"
 		(at 121.92 30.48 90)
@@
 		)
 	)
-	(label "R1"
-		(at 78.74 63.5 180)
-		(effects
-			(font
-				(size 1.27 1.27)
-			)
-			(justify right bottom)
-		)
-	)
 	(label "gSPI_CS"
 		(at 236.22 82.55 270)
@@
 		)
 	)
-	(label "SQ"
-		(at 78.74 55.88 180)
-		(effects
-			(font
-				(size 1.27 1.27)
-			)
-			(justify right bottom)
-		)
-	)
 	(label "UP"
-		(at 96.52 30.48 90)
-		(effects
-			(font
-				(size 1.27 1.27)
-			)
-			(justify left bottom)
+		(at 78.74 40.64 180)
+		(effects
+			(font
+				(size 1.27 1.27)
+			)
+			(justify right bottom)
 		)
 	)
@@
 		(effects
 			(font
-				(size 1.27 1.27)
-			)
-			(justify right bottom)
-		)
-	)
-	(label "X"
-		(at 78.74 43.18 180)
-		(effects
-			(font
